File: pipod_hw.kicad_pcb (KiCad board)
At the start: 4 copper layers, 55.5 x 96.8 mm, 139 parts, among them J1 Conn_01x03_Male, J2 USB_C_Receptacle_USB2.0, J3 SFV8R-2STE1HLF, J4 SFV14R-2STE1HLF, J5 2-1734839-0, J6 2-1734839-0, Q1 DMG9926UDM, Q2 NTK3139PT1G, Q3 BSS138, U1 MAX17048G+T10, U10 TPS22965TDSGRQ1, U11 TPS22965TDSGRQ1, U12 TPS22965TDSGRQ1, U13 PCM5102APWR, U14 PAM8908JER, U15 MCP23008-E/ML, U2 MAX8903AETI+T, U3 BQ29728DSER, U4 XC6210B332MR, U5 W25Q128JVS, U6 RP2040, U7 NLAS7242MUTBG, U8 RS2299XTQC16, U9 TPS22965TDSGRQ1, Y1 12MHz 20pF

Commit message: routing: begin routing
Parts:
- removed J6: 2-1734839-0, Gigahawk:2-1734839-0
- J5: value 2-1734839-0 -> 2-1734839-5; footprint Gigahawk:2-1734839-0 -> Gigahawk:217348395
- moved C28 111.0 mm to (2.80, 22.1)
- moved R36 104.9 mm to (2.08, 23.7), turned to -90 degrees
- moved C31 103.4 mm to (6.36, 24.8), turned to 90 degrees
- moved R35 72.9 mm to (34.6, 37.7)
- moved C27 71.9 mm to (34.6, 36.7)
- moved C30 68.7 mm to (39.4, 38.5), turned to 90 degrees
- moved U10 59.1 mm to (37.2, 37.5)
- moved R44 57.2 mm to (19.1, 10.6), turned to 90 degrees
- moved R43 57.1 mm to (18.6, 12.1), turned to 180 degrees
- moved C32 35.5 mm to (39.8, 37.0), turned to 180 degrees
- moved C33 27.2 mm to (4.71, 22.1), turned to 0 degrees
- moved TP3 13.3 mm to (34.9, 23.3)
- moved TP2 13.2 mm to (33.2, 25.3)
- moved J5 6.45 mm to (41.8, 26.1)
- moved C13 0.35 mm to (29.1, 32.8)
Connections:
- J5 pad 1: GND -> PI_VCC
- J5 pad 10: HP_SL_VIDEO -> PI_USB_MUXED_D+
- J5 pad 11: SMC_PI_I2C_SDA -> SMC_INT
- J5 pad 12: SMC_PI_I2C_SCL -> SMC_TX_PI_RX
- J5 pad 13: SMC_TX_PI_RX -> SMC_RX_PI_TX
- J5 pad 14: SMC_RX_PI_TX -> SMC_PI_I2C_SCL
- J5 pad 15: SMC_INT -> SMC_PI_I2C_SDA
- J5 pad 16: PI_USB_MUXED_D+ -> HP_SL_VIDEO
- J5 pad 17: PI_USB_MUXED_D- -> PI_DISP_SCK
- J5 pad 18: GND -> PI_DISP_MOSI
- J5 pad 19: GND -> PI_DISP_DC
- J5 pad 2: GND -> PI_VCC
- J5 pad 20: GND -> PI_DISP_RST
- J5 pad 3: PI_I2S_BCK -> PI_VCC
- J5 pad 4: PI_I2S_DIN -> PI_VCC
- J5 pad 5: PI_I2S_LRCK -> PI_VCC
- J5 pad 6: PI_DISP_RST -> GND
- J5 pad 7: PI_DISP_DC -> GND
- J5 pad 8: PI_DISP_MOSI -> GND
- J5 pad 9: PI_DISP_SCK -> PI_USB_MUXED_D-
- U6 pad 17: DISP_INPUT_SEL -> unconnected-(U6-Pad17)
- U6 pad 18: SMC_DISP_BL -> unconnected-(U6-Pad18)
- U6 pad 39: unconnected-(U6-Pad39) -> DISP_INPUT_SEL
- U6 pad 40: unconnected-(U6-Pad40) -> SMC_DISP_BL
- U8 pad 1: SMC_DISP_RST -> SMC_DISP_DC
- U8 pad 15: PI_DISP_RST -> PI_DISP_DC
- U8 pad 16: DISP_RST -> DISP_DC
- U8 pad 3: PI_DISP_DC -> PI_DISP_MOSI
- U8 pad 4: DISP_DC -> DISP_MOSI
- U8 pad 5: SMC_DISP_DC -> SMC_DISP_MOSI
- U8 pad 7: PI_DISP_MOSI -> PI_DISP_RST
- U8 pad 8: DISP_MOSI -> DISP_RST
- U8 pad 9: SMC_DISP_MOSI -> SMC_DISP_RST
Routing:
- net GND: track 83.4 -> 170.8 mm, vias 39 -> 84
- net SMC_PI_I2C_SDA: track 0.00 -> 58.5 mm, vias 0 -> 4
- net SMC_PI_I2C_SCL: track 0.00 -> 55.4 mm, vias 0 -> 4
- net PI_USB_MUXED_D-: track 1.32 -> 48.3 mm
- net PI_USB_MUXED_D+: track 1.33 -> 48.3 mm
- net VCC: track 96.3 -> 142.9 mm, vias 5 -> 9
- net PI_DISP_MOSI: track 0.00 -> 36.9 mm, vias 0 -> 2
- net PI_DISP_DC: track 0.00 -> 36.6 mm, vias 0 -> 2
- net PI_DISP_RST: track 0.00 -> 33.8 mm, vias 0 -> 4
- net PI_DISP_SCK: track 0.00 -> 32.9 mm, vias 0 -> 3
- net SMC_DISP_DC: track 0.00 -> 30.1 mm, vias 0 -> 3
- net PI_VCC_EN: track 1.23 -> 29.5 mm, vias 0 -> 4
- net DISP_3V3_EN: track 1.24 -> 27.4 mm, vias 1 -> 6
- net SMC_DISP_BL: track 0.00 -> 26.1 mm, vias 0 -> 2
- net SMC_DISP_SCK: track 0.00 -> 25.8 mm, vias 0 -> 3
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