File: audio.kicad_sch (KiCad schematic)
At the start: 27 parts, among them U13 PCM5102APWR, U14 PAM8908JER

Commit message: ci: prepare files for CI
Parts:
- U14: footprint Package_DFN_QFN:QFN-16-1EP_3x3mm_P0.5mm_EP1.7x1.7mm -> Gigahawk:QFN-16-1EP_3x3mm_P0.5mm_EP1.7x1.7mm
Other:
- title: (none) -> piPod IO/SMC Board
Changed lines of the file:
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@@
 (kicad_sch (version 20211123) (generator eeschema)
   (paper "A4")
+  (title_block
+    (title "piPod IO/SMC Board")
+    (date "${DATE}")
+    (rev "%{TAG} (${REVISION})")
+  )
   (junction (at 78.74 130.81) (diameter 0) (color 0 0 0 0)
   )
@@
     (property "Reference" "U14" (id 0) (at 222.25 54.61 0))
     (property "Value" "PAM8908JER" (id 1) (at 233.68 88.9 0))
-    (property "Footprint" "Package_DFN_QFN:QFN-16-1EP_3x3mm_P0.5mm_EP1.7x1.7mm" (id 2) (at 222.25 91.44 0)
-      (effects (font (size 1.27 1.27)) hide)
-    )
+    (property "Footprint" "Gigahawk:QFN-16-1EP_3x3mm_P0.5mm_EP1.7x1.7mm" (id 2) (at 222.25 91.44 0)
+      (effects (font (size 1.27 1.27)) hide)
+    )
